File: Schaltplan.sch (EAGLE design)
At the start: 58 parts, among them Q1 TN0602N3, Q10 TN0602N3, Q11 TN0602N3, Q12 TN0602N3, Q13 TN0602N3, Q14 TN0602N3, Q15 TN0602N3, Q16 TN0602N3, Q17 TN0602N3, Q18 TN0602N3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

Commit message: Fixed Bug: Missing connection
Parts:
- removed U$1, U$2: LOGO, logo:LOGO
Changed lines of the file:
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@@
 <part name="GND27" library="supply1" deviceset="GND" device=""/>
 <part name="GND28" library="supply1" deviceset="GND" device=""/>
-<part name="U$1" library="logo" deviceset="LOGO" device=""/>
-<part name="U$2" library="logo" deviceset="LOGO" device=""/>
 <part name="U$3" library="logo" deviceset="LOGO" device=""/>
 </parts>
@@
 <wire x1="60.96" y1="101.6" x2="66.04" y2="101.6" width="0.1524" layer="91"/>
 <wire x1="66.04" y1="101.6" x2="66.04" y2="129.54" width="0.1524" layer="91"/>
+<junction x="60.96" y="101.6"/>
+<label x="86.36" y="129.54" size="1.778" layer="95"/>
 <pinref part="Q15" gate="G$1" pin="G"/>
 <wire x1="200.66" y1="129.54" x2="66.04" y2="129.54" width="0.1524" layer="91"/>
-<junction x="60.96" y="101.6"/>
-<label x="86.36" y="129.54" size="1.778" layer="95"/>
 </segment>
 </net>
